File: beelight-piggy-base/beelight-piggy-base.kicad_sch (KiCad schematic)
At the start: 85 parts, among them J1 B_Le, J2 B_Ri, J3 USB_C_Receptacle_PowerOnly_6P, J4 WS2812_ext, J5 Conn_01x07_Pin, J6 BatSide, J7 DevSide, J8 B_Ri, J9 B_Le, Q1 AO3400A, SW1 SW_Push, U2 BMA253, U3 TPS22917LDBV, U4 rysta, U5 VEML3328, U6 TSOP382xx, U7 MP2667, U8 BQ27421-G1

Commit message: fix usb-c input cc resistors
Parts:
- removed J3: USB_C_Receptacle_PowerOnly_6P, Connector_USB:USB_C_Receptacle_GCT_USB4125-xx-x-0190_6P_TopMnt_Horizontal, symbol Connector:USB_C_Receptacle_PowerOnly_6P
- added J10: USB C power only, .local:USB_C_Receptacle_GCT_USB4125-xx-x_6P_TopMnt_Horizontal, symbol .local:USB_C_Receptacle_PowerOnly_6P
- D23, D24, D25, D26: value Schottky -> tbd
- R1, R2: value 22k -> 5k1
- R21, R22: value 100k -> 100k tbd
Connections:
- net GND: now also R1.2, R2.1, J10.A12 (GND), J10.B12 (GND), J10.SH (SHIELD)
- net VBUS: now also J10.A9 (VBUS), J10.B9 (VBUS); no longer R1.1, R2.1
- net at R2.2: now also J10.B5 (CC2)
- new net: J10.A5 (CC1), R1.1
Other:
- moved on the sheet: C1, C25, C26, C27, C28, C29, D24, D25, D26, R1, R18, R19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
