File: beelight-piggy-base/beelight-piggy-base.kicad_sch (KiCad schematic)
At the start: 74 parts, among them J1 B_Le, J10 USB C power only, J11 ExtWSSolderPads, J2 B_Ri, J3 BatSolderPads, J4 WS2812_ext, J5 Conn_01x07_Pin, J6 BatSide, J7 DevSide, J8 B_Ri, J9 B_Le, Q1 AO3400A, SW1 SW_Push, U2 BMA253, U3 TPS22917LDBV, U4 rysta, U5 VEML3328, U6 TSOP382xx, U7 MP2667, U8 BQ27421-G1

Commit message: pre-optimize
Parts:
- C27: value 1uF -> 2.2uF
- U8: value BQ27421-G1 -> bq27427yzfr
Changed lines of the file:
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@@
 			)
 		)
-		(property "Value" "BQ27421-G1"
+		(property "Value" "bq27427yzfr"
 			(at 148.59 220.98 0)
 			(show_name no)
@@
 			)
 		)
-		(property "Value" "1uF"
+		(property "Value" "2.2uF"
 			(at 168.91 246.3799 0)
 			(show_name no)
