File: beelight-piggy-base/beelight-piggy-base.kicad_pcb (KiCad board)
At the start: 2 copper layers, 55 x 55 mm, 67 parts, among them J10 USB C power only, J11 ExtWSSolderPads, J3 BatSolderPads, J4 WS2812_ext, J7 DevSide, Q1 AO3400A, SW1 SW_Push, U2 BMA253, U3 TPS22917LDBV, U4 rysta, U5 VEML3328, U6 TSOP382xx, U7 MP2667, U8 BQ27421-G1

Commit message: pre-optimize
Parts:
- C27: value 1uF -> 2.2uF
- U8: value BQ27421-G1 -> bq27427yzfr
Changed lines of the file:
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@@
 			)
 		)
-		(property "Value" "1uF"
+		(property "Value" "2.2uF"
 			(at 0 1.16 90)
 			(layer "F.Fab")
@@
 			)
 		)
-		(property "LCSC" "C52923"
+		(property "LCSC" "C170151"
 			(at 0 0 0)
 			(layer "F.SilkS")
@@
 			)
 		)
+		(property "LCSC" "C15850"
+			(at 0 0 0)
+			(layer "F.SilkS")
+			(hide yes)
+			(effects
+				(font
+					(size 1.27 1.27)
+					(thickness 0.15)
+				)
+			)
+		)
 		(property ki_fp_filters "C_*")
 		(sheetname "/")
@@
 			)
 		)
-		(property "Value" "BQ27421-G1"
+		(property "Value" "bq27427yzfr"
 			(at 0 1.95 90)
 			(layer "F.Fab")
@@
 			)
 		)
-		(property "LCSC" "C2871789"
+		(property "LCSC" "C6075475"
 			(at 0 0 0)
 			(layer "F.SilkS")
